File: Levitator.kicad_pcb (KiCad board)
At the start: 2 copper layers, 15 parts, among them P1 POWER, P2 COIL, P3 HC06 SERIAL, P4 SENSOR, P5 BT_SWITCH, Q1 IRL540N

Commit message: Endspurt
Parts:
- removed P1: POWER, Connector_JST:JST_EH_B2B-EH-A_1x02_P2.50mm_Vertical
- removed P2: COIL, Connector_JST:JST_EH_B2B-EH-A_1x02_P2.50mm_Vertical
- removed P3: HC06 SERIAL, Connector_JST:JST_EH_B4B-EH-A_1x04_P2.50mm_Vertical
- removed P4: SENSOR, Connector_JST:JST_EH_B3B-EH-A_1x03_P2.50mm_Vertical
- removed P5: BT_SWITCH, digikey-footprints:PinHeader_1x2_P2.54mm_Drill1.02mm
- added B1: HC-06, nrth3rnlb-footprints:HC-06, F.Cu at (166.2, 72.8)
- added C3: 1m, Capacitor_THT:C_Rect_L7.0mm_W3.5mm_P2.50mm_P5.00mm, F.Cu at (185.8, 115.2)
- added C4: 220n, Capacitor_THT:C_Rect_L7.0mm_W3.5mm_P2.50mm_P5.00mm, F.Cu at (178.8, 115.2)
- added C6: 100n, Capacitor_THT:C_Rect_L7.0mm_W3.5mm_P2.50mm_P5.00mm, F.Cu at (171.8, 115.2)
- added H1: MountingHole, MountingHole:MountingHole_3.2mm_M3, F.Cu at (185.3, 125.7)
- added H2: MountingHole, MountingHole:MountingHole_3.2mm_M3, F.Cu at (132.3, 72.7)
- added H3: MountingHole, MountingHole:MountingHole_3.2mm_M3, F.Cu at (132.3, 125.7)
- added H4: MountingHole, MountingHole:MountingHole_3.2mm_M3, F.Cu at (185.3, 72.7)
- added J1: POWER, Connector_JST:JST_EH_B2B-EH-A_1x02_P2.50mm_Vertical, F.Cu at (142.9, 129.6)
- added J2: SENSOR, Connector_JST:JST_EH_B3B-EH-A_1x03_P2.50mm_Vertical, F.Cu at (142.9, 118.8)
- added J3: BT_ON, Connector_JST:JST_EH_B2B-EH-A_1x02_P2.50mm_Vertical, F.Cu at (176.1, 69.0)
- added J4: COIL, Connector_JST:JST_EH_B2B-EH-A_1x02_P2.50mm_Vertical, F.Cu at (177.9, 125.9)
- added NT1: Net-Tie_3, NetTie:NetTie-3_THT_Pad1.0mm, F.Cu at (166.8, 121.2)
- added REF**: KiCad-Logo2_5mm_SilkScreen, Symbol:KiCad-Logo2_5mm_SilkScreen, F.Cu at (158.8, 135.2)
- added U1: DC-DC_Regulator, nrth3rnlb-footprints:Board_45x20, F.Cu at (179.8, 72.4)
- added U2: MC7805CT-BP, Package_TO_SOT_THT:TO-220-3_Horizontal_TabDown, F.Cu at (171.6, 96.6)
- A1: value Arduino_Nano_v2.x -> Arduino_Nano_v2
- C5: value C -> 100n
- D2: value LED -> COIL
- Q1: footprint Package_TO_SOT_THT:TO-220-3_Vertical -> Package_TO_SOT_THT:TO-220-3_Horizontal_TabDown
- moved D1 87.1 mm to (171.0, 124.3), turned to 270 degrees
- moved C5 77.7 mm to (151.7, 101.5), turned to 90 degrees
- moved Q1 72.6 mm to (161.4, 112.2), turned to 180 degrees
- moved A1 62.0 mm to (159.4, 91.6)
- moved D3 61.4 mm to (165.2, 63.5)
- moved D2 59.8 mm to (155.6, 63.5)
- moved R2 58.7 mm to (162.6, 69.9), turned to 0 degrees
- moved R1 52.7 mm to (148.0, 69.9), turned to 0 degrees
- moved C2 52.4 mm to (131.4, 96.5), turned to 270 degrees
- moved C1 46.4 mm to (131.5, 116.2), turned to 90 degrees
Connections:
- A1 pad 27: +5V -> Net-(A1-Pad27)
Other:
- board outline added: 80 x 80 mm
- board text added: "7805"
- board text added: "7805 OR DC-DC Regulator"
- board text added: "Levitator"

Commit message: add gerber
Routing:
- net GND: track 0.00 -> 201.3 mm
- net VIN: track 0.00 -> 129.9 mm
- net +5V: track 0.00 -> 80.1 mm
- net COIL_CTRL: track 0.00 -> 67.9 mm
- net Net-(A1-Pad11): track 0.00 -> 37.7 mm
- net Net-(D1-Pad2): track 0.00 -> 33.2 mm
- net SENSOR: track 0.00 -> 28.3 mm
- net Net-(A1-Pad18): track 0.00 -> 25.2 mm
- net +5V_2: track 0.00 -> 22.5 mm
- net +5V_1: track 0.00 -> 19.7 mm
- net Net-(B1-Pad1): track 0.00 -> 15.8 mm
- net TX: track 0.00 -> 11.2 mm
- net Net-(D3-Pad2): track 0.00 -> 10.9 mm
- net RX: track 0.00 -> 9.66 mm
- net Net-(D2-Pad2): track 0.00 -> 7.40 mm

Commit message: done
Parts:
- added OpenHardware: OSHW-Logo2_7.3x6mm_SilkScreen, Symbol:OSHW-Logo2_7.3x6mm_SilkScreen, F.Cu at (142.2, 67.9)
- J3: value BT_ON -> BT_SWITCH
- moved B1 37.8 mm to (132.1, 88.9), turned to 90 degrees
- moved NT1 15.6 mm to (182.3, 119.9), turned to 180 degrees
Connections:
- A1 pad 10: Net-(A1-Pad10) -> (no net)
- A1 pad 13: Net-(A1-Pad13) -> (no net)
- A1 pad 14: Net-(A1-Pad14) -> (no net)
- A1 pad 15: Net-(A1-Pad15) -> (no net)
- A1 pad 16: Net-(A1-Pad16) -> (no net)
- A1 pad 17: Net-(A1-Pad17) -> (no net)
- A1 pad 20: Net-(A1-Pad20) -> (no net)
- A1 pad 21: Net-(A1-Pad21) -> (no net)
- A1 pad 22: Net-(A1-Pad22) -> (no net)
- A1 pad 23: Net-(A1-Pad23) -> (no net)
- A1 pad 24: Net-(A1-Pad24) -> (no net)
- A1 pad 25: Net-(A1-Pad25) -> (no net)
- A1 pad 26: Net-(A1-Pad26) -> (no net)
- A1 pad 27: Net-(A1-Pad27) -> (no net)
- A1 pad 28: Net-(A1-Pad28) -> (no net)
- A1 pad 3: Net-(A1-Pad3) -> (no net)
- A1 pad 5: Net-(A1-Pad5) -> (no net)
- A1 pad 6: Net-(A1-Pad6) -> (no net)
- A1 pad 7: Net-(A1-Pad7) -> (no net)
- A1 pad 8: Net-(A1-Pad8) -> (no net)
- A1 pad 9: Net-(A1-Pad9) -> (no net)
Routing:
- net Net-(B1-Pad1): track 15.8 -> 50.7 mm
- net RX: track 9.66 -> 33.7 mm
- net TX: track 11.2 -> 28.6 mm
- net +5V_2: track 22.5 -> 6.62 mm
- net GND: track 201.3 -> 217.1 mm
- net +5V: track 80.1 -> 92.8 mm
- net VIN: track 129.9 -> 132.7 mm
- net +5V_1: track 19.7 -> 21.9 mm
- net COIL_CTRL: track 67.9 -> 67.0 mm
- net Net-(D3-Pad2): track 10.9 -> 10.3 mm
- added copper zone on B.Cu, net GND
- added copper zone on F.Cu, net GND
Other:
- board text added: "https://github.com/aboettger/levitator"
