File: Levitator.sch (KiCad schematic (older format))
At the start: 19 parts

Commit message: foobar
Parts:
- removed C?: CP, symbol Device:CP
- added C3: 220nF, Capacitor_THT:C_Rect_L7.0mm_W2.5mm_P5.00mm, symbol Device:C
- added C6: 1mF, Capacitor_THT:C_Rect_L7.0mm_W2.5mm_P5.00mm, symbol Device:C
- C1: renamed from C?; value CP -> 1000uF; footprint (none) -> Capacitor_THT:CP_Radial_D8.0mm_P3.50mm
- C2, C4: renamed from C?; value C -> 100nF; footprint (none) -> Capacitor_THT:C_Rect_L7.0mm_W2.5mm_P5.00mm
- C5: renamed from C?; footprint (none) -> Capacitor_THT:C_Rect_L7.0mm_W2.5mm_P5.00mm
- D2, D3: renamed from D?; footprint (none) -> LED_THT:LED_D3.0mm
- J2: renamed from J?; footprint (none) -> Connector_JST:JST_EH_B3B-EH-A_1x03_P2.50mm_Vertical
- R1, R2: renamed from R?; value R -> 330; footprint (none) -> Resistor_THT:R_Axial_DIN0204_L3.6mm_D1.6mm_P7.62mm_Horizontal
- gave numbers to parts that had none: 9
Connections:
- net +5V: no longer A1.27 (+5V)
- net EXT_Reg: now also C3.1, C6.1
- net GND: now also C3.2, C6.2
- no-connect marks 0 -> 22
Other:
- moved on the sheet: C4, U1

Commit message: Endspurt
Parts:
- removed J3: HC06 SERIAL, symbol Connector_Generic:Conn_01x04
- removed JP1, JP2: Jumper_3_Open, symbol Jumper:Jumper_3_Open
- removed U1: LM7805_TO220, Package_TO_SOT_THT:TO-220-3_Vertical, symbol Regulator_Linear:LM7805_TO220
- added B1: HC-06, nrth3rnlb-footprints:HC-06, symbol nrth3rnlb_Bluetooth-Modules:HC-06
- added H1, H2, H3, H4: MountingHole, MountingHole:MountingHole_3.2mm_M3, symbol Mechanical:MountingHole
- added J3: BT_ON, Connector_JST:JST_EH_B2B-EH-A_1x02_P2.50mm_Vertical, symbol dk_Rectangular-Connectors-Headers-Male-Pins:22-23-2021
- added NT1: Net-Tie_3, NetTie:NetTie-3_THT_Pad1.0mm, symbol Device:Net-Tie_3
- added U1: DC-DC_Regulator, nrth3rnlb-footprints:Board_45x20, symbol nrth3rnlb_DCDC-Modules:DC-DC_Regulator
- added U2: MC7805CT-BP, Package_TO_SOT_THT:TO-220-3_Horizontal_TabDown, symbol dk_PMIC-Voltage-Regulators-Linear:MC7805CT-BP
- A1: value Arduino_Nano_v2.x -> Arduino_Nano_v2
- C3: value 220nF -> 1m; footprint Capacitor_THT:C_Rect_L7.0mm_W2.5mm_P5.00mm -> Capacitor_THT:C_Rect_L7.0mm_W3.5mm_P2.50mm_P5.00mm
- C4: value 100nF -> 220n; footprint Capacitor_THT:C_Rect_L7.0mm_W2.5mm_P5.00mm -> Capacitor_THT:C_Rect_L7.0mm_W3.5mm_P2.50mm_P5.00mm
- C5: value C -> 100n
- C6: value 1mF -> 100n; footprint Capacitor_THT:C_Rect_L7.0mm_W2.5mm_P5.00mm -> Capacitor_THT:C_Rect_L7.0mm_W3.5mm_P2.50mm_P5.00mm
- D2: value LED -> COIL
- J1, J4: footprint digikey-footprints:PinHeader_1x2_P2.54mm_Drill1.02mm -> Connector_JST:JST_EH_B2B-EH-A_1x02_P2.50mm_Vertical
- J2: symbol Connector_Generic:Conn_01x03 -> dk_Rectangular-Connectors-Headers-Male-Pins:640456-3
- Q1: footprint Package_TO_SOT_THT:TO-220-3_Vertical -> Package_TO_SOT_THT:TO-220-3_Horizontal_TabDown
Connections:
- net POWER is gone; now on net VIN: C1.1, D1.1 (K), J1.1, J4.1
- net +5V: now also J3.1, NT1.2; no longer C4.1
- net GND: now also B1.2 (GND), U1.2 (IN-), U1.4 (OUT-), U2.2 (GND)
- net RX: now also B1.4 (RX)
- net TX: now also B1.3 (TX)
- net VIN: now also C3.1, C4.1, U1.1 (IN+), U2.1 (IN)
- net EXT_Reg renamed +5V_1
- net +5V_1: now also NT1.3, U2.3 (OUT); no longer C3.1
- new net: B1.1 (VCC), J3.2
- new net +5V_2: NT1.1, U1.3 (OUT+)
- no-connect marks 22 -> 21
Other:
- note removed: "if power supply < 15V"
- note removed: "if power supply >= 15V"
- moved on the sheet: A1, C5, D3, R2

Commit message: done
Parts:
- J3: value BT_ON -> BT_SWITCH
Changed lines of the file:
@@
 P 1450 6700
 F 0 "J3" V 1350 6650 50  0000 C CNN
-F 1 "BT_ON" H 1500 6550 50  0000 C CNN
+F 1 "BT_SWITCH" H 1500 6550 50  0000 C CNN
 F 2 "Connector_JST:JST_EH_B2B-EH-A_1x02_P2.50mm_Vertical" H 1650 6900 60  0001 L CNN
 F 3 "https://media.digikey.com/pdf/Data%20Sheets/Molex%20PDFs/A-6373-N_Series_Dwg_2010-12-03.pdf" H 1650 7000 60  0001 L CNN
@@
 	1    0    0    -1
 $EndComp
+$Comp
+L power:PWR_FLAG #FLG0101
+U 1 1 5ED74AAA
+P 1550 6800
+F 0 "#FLG0101" H 1550 6875 50  0001 C CNN
+F 1 "PWR_FLAG" H 1550 6973 50  0000 C CNN
+F 2 "" H 1550 6800 50  0001 C CNN
+F 3 "~" H 1550 6800 50  0001 C CNN
+	1    1550 6800
+	0    1    1    0
+$EndComp
+Connection ~ 1550 6800
 $EndSCHEMATC
